File: PCB/Leiterkarte-v2.kicad_sch (KiCad schematic)
At the start: 39 parts

Commit message: Replaced Fuse;Updated BOM file
Parts:
- F1: value 1.5A -> 2A; footprint Fuse:0458Series_LTF-M -> Fuse:Fuse_1206_3216Metric
Changed lines of the file:
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@@
 			)
 		)
-		(property "Value" "1.5A"
+		(property "Value" "2A"
 			(at 35.306 27.94 90)
 			(effects
@@
 			)
 		)
-		(property "Footprint" "Fuse:0458Series_LTF-M"
+		(property "Footprint" "Fuse:Fuse_1206_3216Metric"
 			(at 35.306 27.94 90)
 			(effects

Commit message: Added pulldown resistors for the buttons;Changed input GPIof button 3;Replaced a few capacitors (BOM); Put temperature sensors on the 3.3V line
Parts:
- added Rbtn1, Rbtn2, Rbtn3: 10k, Resistor_SMD:R_0603_1608Metric, symbol Device:R
- Cin2: value 10uF -> 1uF
- Cout1: value 22uF -> 2.2uF
Connections:
- net +3.3V: now also TEMP_S1.1 (V_{DD}), TEMP_S2.3 (Pin_3)
- net +5V: no longer TEMP_S1.1 (V_{DD}), TEMP_S2.3 (Pin_3)
- net Button1: now also Rbtn1.1
- net Button2: now also Rbtn2.1
- net Button3: now also Rbtn3.2
- net GND: now also Rbtn1.2, Rbtn2.2, Rbtn3.1
Other:
- note added: "RPM Out: Square 2.4-3V"
- note removed: "RPM Out: Square 3V"
- moved on the sheet: Buttons1, Fan1, Qfan1

Commit message: Initializing Firmware Project
Parts:
- renumbered Rbtn3 to Rbtn2, Rbtn2 to Rbtn3, TEMP_S2 to TEMP_S1, TEMP_S1 to TEMP_S2, 3.3V1 to V3.31
